File: Bad Apple.kicad_pcb (KiCad board)
At the start: 2 copper layers, 65 x 56 mm, 5 parts, among them J1 GPIO

Commit message: chore: dummy PCB thingymabob
Parts:
- added C1: 100n, Capacitor_SMD:C_0805_2012Metric, F.Cu at (163.0, 61.5)
- added D1: D, Diode_SMD:D_SOD-323F, F.Cu at (137.0, 66.2)
- added H1: MountingHole, MountingHole:MountingHole_2.2mm_M2, F.Cu at (52.8, 44.4)
- added H2: MountingHole, MountingHole:MountingHole_2.2mm_M2, F.Cu at (58.1, 44.4)
- added H3: MountingHole, MountingHole:MountingHole_2.2mm_M2, F.Cu at (63.5, 44.4)
- added H4: MountingHole, MountingHole:MountingHole_2.2mm_M2, F.Cu at (69.0, 44.0)
- added J10: Conn_01x04, Connector_PinHeader_2.54mm:PinHeader_1x04_P2.54mm_Vertical, F.Cu at (111.8, 63.6)
- added J11: Conn_01x03, Connector_PinHeader_2.54mm:PinHeader_1x03_P2.54mm_Vertical, F.Cu at (158.0, 87.9)
- added J12: Conn_01x03, Connector_PinHeader_2.54mm:PinHeader_1x03_P2.54mm_Vertical, F.Cu at (157.9, 91.5)
- added J2: Conn_01x02, Connector_Wire:SolderWire-0.1sqmm_1x02_P3.6mm_D0.4mm_OD1mm, F.Cu at (125.5, 75.8)
- added J3: Conn_01x02, Connector_Wire:SolderWire-0.1sqmm_1x02_P3.6mm_D0.4mm_OD1mm, F.Cu at (102.0, 86.0)
- added J4: Conn_01x02, Connector_Wire:SolderWire-0.1sqmm_1x02_P3.6mm_D0.4mm_OD1mm, F.Cu at (105.5, 86.0)
- added J5: Conn_01x02, Connector_Wire:SolderWire-0.1sqmm_1x02_P3.6mm_D0.4mm_OD1mm, F.Cu at (102.0, 88.7)
- added J6: Conn_01x02, Connector_Wire:SolderWire-0.1sqmm_1x02_P3.6mm_D0.4mm_OD1mm, F.Cu at (105.5, 88.7)
- added J7: Conn_01x04, Connector_PinHeader_2.54mm:PinHeader_1x04_P2.54mm_Vertical, F.Cu at (116.5, 63.4)
- added J9: Conn_01x04, Connector_PinHeader_2.54mm:PinHeader_1x04_P2.54mm_Vertical, F.Cu at (107.2, 63.6)
- added JP1: ID_WP, Jumper:SolderJumper-2_P1.3mm_Open_RoundedPad1.0x1.5mm, F.Cu at (160.3, 56.8)
- added JP2: SolderJumper_2_Open, Jumper:SolderJumper-2_P1.3mm_Open_RoundedPad1.0x1.5mm, F.Cu at (135.5, 98.0)
- added JP3: SolderJumper_2_Open, Jumper:SolderJumper-2_P1.3mm_Open_RoundedPad1.0x1.5mm, F.Cu at (139.1, 98.0)
- added JP4: SolderJumper_2_Open, Jumper:SolderJumper-2_P1.3mm_Open_RoundedPad1.0x1.5mm, F.Cu at (142.6, 98.0)
- added JP5: SolderJumper_2_Open, Jumper:SolderJumper-2_P1.3mm_Open_RoundedPad1.0x1.5mm, F.Cu at (146.2, 98.0)
- added JP6: SolderJumper_2_Open, Jumper:SolderJumper-2_P1.3mm_Open_RoundedPad1.0x1.5mm, F.Cu at (149.7, 98.0)
- added JP7: SolderJumper_2_Open, Jumper:SolderJumper-2_P1.3mm_Open_RoundedPad1.0x1.5mm, F.Cu at (153.2, 98.0)
- added Q1: SS8050, Package_TO_SOT_SMD:SOT-23, F.Cu at (134.2, 64.5)
- added R1: 3.9k, Resistor_SMD:R_1206_3216Metric, F.Cu at (144.2, 52.8)
- added R10: R, Resistor_SMD:R_0805_2012Metric, F.Cu at (139.4, 64.0)
- added R2: 3.9k, Resistor_SMD:R_1206_3216Metric, F.Cu at (147.8, 52.8)
- added R3: R, Resistor_SMD:R_0805_2012Metric, F.Cu at (136.7, 93.7)
- added R4: R, Resistor_SMD:R_0805_2012Metric, F.Cu at (139.7, 93.7)
- added R5: R, Resistor_SMD:R_0805_2012Metric, F.Cu at (142.6, 93.7)
- added R6: R, Resistor_SMD:R_0805_2012Metric, F.Cu at (145.6, 93.7)
- added R7: R, Resistor_SMD:R_0805_2012Metric, F.Cu at (148.5, 93.7)
- added R8: R, Resistor_SMD:R_0805_2012Metric, F.Cu at (151.4, 93.7)
- added R9: R, Resistor_SMD:R_0805_2012Metric, F.Cu at (65.8, 108.2)
- added U1: CAT24C256, Package_SO:SOIC-8_3.9x4.9mm_P1.27mm, F.Cu at (139.6, 56.2)
- added U2: ICM-20948, Sensor_Motion:InvenSense_QFN-24_3x3mm_P0.4mm, F.Cu at (103.9, 56.5)
- added U3: TXS0104EPW, Package_SO:TSSOP-14_4.4x5mm_P0.65mm, F.Cu at (111.1, 56.4)
- added U4: PCA9685BS, Package_DFN_QFN:QFN-28-1EP_6x6mm_P0.65mm_EP4.25x4.25mm, F.Cu at (157.9, 70.5)
- added U5: TB6612FNG, Package_SO:SSOP-24_5.3x8.2mm_P0.65mm, F.Cu at (113.0, 88.4)
- added U6: TB6612FNG, Package_SO:SSOP-24_5.3x8.2mm_P0.65mm, F.Cu at (124.2, 94.2)
Connections:
- net /GPIO14/TXD0 renamed /[1] HAT Interface/GPIO14/TXD0
- net /GPIO16 renamed /[1] HAT Interface/GPIO16
- net /GPIO20/PCM.DIN renamed /[1] HAT Interface/GPIO20/PCM.DIN
- net /GPIO21/PCM.DOUT renamed /[1] HAT Interface/GPIO21/PCM.DOUT
- net /GPIO23 renamed /[1] HAT Interface/GPIO23
- net /GPIO24 renamed /[1] HAT Interface/GPIO24
- net /GPIO25 renamed /[1] HAT Interface/GPIO25
- net /GPIO26 renamed /[1] HAT Interface/GPIO26
- net /GPIO4/GPCLK0 renamed /[1] HAT Interface/GPIO4/GPCLK0
- net /GPIO8/SPI0.CE0 renamed /[1] HAT Interface/GPIO8/SPI0.CE0
- J1 pad 10: /GPIO15/RXD0 -> /[1] HAT Interface/GPIO15/RXD0
- J1 pad 11: /GPIO17 -> /[1] HAT Interface/GPIO17
- J1 pad 12: /GPIO18/PCM.CLK -> /[1] HAT Interface/GPIO18/PCM.CLK
- J1 pad 13: /GPIO27 -> /[1] HAT Interface/GPIO27
- J1 pad 15: /GPIO22 -> /[1] HAT Interface/GPIO22
- J1 pad 19: /GPIO10/SPI0.MOSI -> /[1] HAT Interface/GPIO10/SPI0.MOSI
- J1 pad 21: /GPIO9/SPI0.MISO -> /[1] HAT Interface/GPIO9/SPI0.MISO
- J1 pad 23: /GPIO11/SPI0.SCLK -> /[1] HAT Interface/GPIO11/SPI0.SCLK
- J1 pad 26: /GPIO7/SPI0.CE1 -> /[1] HAT Interface/GPIO7/SPI0.CE1
- J1 pad 27: /ID_SDA -> /[1] HAT Interface/ID_SDA
- J1 pad 28: /ID_SCL -> /[1] HAT Interface/ID_SCL
- J1 pad 29: /GPIO5 -> /[1] HAT Interface/GPIO5
- J1 pad 3: /GPIO2/SDA1 -> /[1] HAT Interface/GPIO2/SDA1
- J1 pad 31: /GPIO6 -> /[1] HAT Interface/GPIO6
- J1 pad 32: /GPIO12/PWM0 -> /[1] HAT Interface/GPIO12/PWM0
- J1 pad 33: /GPIO13/PWM1 -> /[1] HAT Interface/GPIO13/PWM1
- J1 pad 35: /GPIO19/PCM.FS -> /[1] HAT Interface/GPIO19/PCM.FS
- J1 pad 5: /GPIO3/SCL1 -> /[1] HAT Interface/GPIO3/SCL1
Routing:
- net /[1] HAT Interface/GPIO19/PCM.FS: track 0.00 -> 71.3 mm, vias 0 -> 3
- net /[1] HAT Interface/GPIO6: track 0.00 -> 70.9 mm, vias 0 -> 1
- net /[1] HAT Interface/GPIO5: track 0.00 -> 67.8 mm, vias 0 -> 3
- net /[1] HAT Interface/GPIO27: track 0.00 -> 63.7 mm, vias 0 -> 2
- net /[1] HAT Interface/GPIO3/SCL1: track 0.00 -> 59.6 mm
- net /[1] HAT Interface/GPIO2/SDA1: track 0.00 -> 59.3 mm
- net /[1] HAT Interface/GPIO17: track 0.00 -> 53.5 mm, vias 0 -> 4
- net /[1] HAT Interface/GPIO7/SPI0.CE1: track 0.00 -> 44.6 mm
- net /[1] HAT Interface/GPIO12/PWM0: track 0.00 -> 44.6 mm
- net /[4] Motors/[4b] Servo Motor Driver/PWM A0: track 0.00 -> 43.4 mm
- net /[4] Motors/[4b] Servo Motor Driver/PWM A1: track 0.00 -> 40.2 mm
- net /[1] HAT Interface/GPIO11/SPI0.SCLK: track 0.00 -> 37.9 mm
- net /[1] HAT Interface/GPIO9/SPI0.MISO: track 0.00 -> 37.5 mm
- net /[4] Motors/[4b] Servo Motor Driver/PWM A2: track 0.00 -> 36.7 mm
- net /[4] Motors/[4b] Servo Motor Driver/PWM A5: track 0.00 -> 36.3 mm, vias 0 -> 4
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Other:
- outline, holes or cut-outs redrawn
- board text added: "CPU Fan"
- board text added: "DC Motors"
- board text added: "Left"
- board text added: "LiDAR Scanner"
- board text added: "PWM Config"
- board text added: "Right"
- board text added: "Write Lock"
- board text removed: "CAMERA (OPTIONAL)"

Commit message: feat: cleared the PCB design for a much better thingy
Parts:
- removed C1: 100n, Capacitor_SMD:C_0805_2012Metric
- removed D1: D, Diode_SMD:D_SOD-323F
- removed H1, H2, H3, H4: MountingHole, MountingHole:MountingHole_2.2mm_M2
- removed J10, J7, J9: Conn_01x04, Connector_PinHeader_2.54mm:PinHeader_1x04_P2.54mm_Vertical
- removed J11, J12: Conn_01x03, Connector_PinHeader_2.54mm:PinHeader_1x03_P2.54mm_Vertical
- removed J2, J3, J4, J5, J6: Conn_01x02, Connector_Wire:SolderWire-0.1sqmm_1x02_P3.6mm_D0.4mm_OD1mm
- removed JP1: ID_WP, Jumper:SolderJumper-2_P1.3mm_Open_RoundedPad1.0x1.5mm
- removed JP2, JP3, JP4, JP5, JP6, JP7: SolderJumper_2_Open, Jumper:SolderJumper-2_P1.3mm_Open_RoundedPad1.0x1.5mm
- removed Q1: SS8050, Package_TO_SOT_SMD:SOT-23
- removed R1, R2: 3.9k, Resistor_SMD:R_1206_3216Metric
- removed R10, R3, R4, R5, R6, R7, R8, R9: R, Resistor_SMD:R_0805_2012Metric
- removed U1: CAT24C256, Package_SO:SOIC-8_3.9x4.9mm_P1.27mm
- removed U2: ICM-20948, Sensor_Motion:InvenSense_QFN-24_3x3mm_P0.4mm
- removed U3: TXS0104EPW, Package_SO:TSSOP-14_4.4x5mm_P0.65mm
- removed U4: PCA9685BS, Package_DFN_QFN:QFN-28-1EP_6x6mm_P0.65mm_EP4.25x4.25mm
- removed U5, U6: TB6612FNG, Package_SO:SSOP-24_5.3x8.2mm_P0.65mm
Connections:
- net /[1] HAT Interface/GPIO14/TXD0 renamed /GPIO14/TXD0
- net /[1] HAT Interface/GPIO16 renamed /GPIO16
- net /[1] HAT Interface/GPIO20/PCM.DIN renamed /GPIO20/PCM.DIN
- net /[1] HAT Interface/GPIO21/PCM.DOUT renamed /GPIO21/PCM.DOUT
- net /[1] HAT Interface/GPIO23 renamed /GPIO23
- net /[1] HAT Interface/GPIO24 renamed /GPIO24
- net /[1] HAT Interface/GPIO25 renamed /GPIO25
- net /[1] HAT Interface/GPIO26 renamed /GPIO26
- net /[1] HAT Interface/GPIO4/GPCLK0 renamed /GPIO4/GPCLK0
- net /[1] HAT Interface/GPIO8/SPI0.CE0 renamed /GPIO8/SPI0.CE0
- J1 pad 10: /[1] HAT Interface/GPIO15/RXD0 -> /GPIO15/RXD0
- J1 pad 11: /[1] HAT Interface/GPIO17 -> /GPIO17
- J1 pad 12: /[1] HAT Interface/GPIO18/PCM.CLK -> /GPIO18/PCM.CLK
- J1 pad 13: /[1] HAT Interface/GPIO27 -> /GPIO27
- J1 pad 15: /[1] HAT Interface/GPIO22 -> /GPIO22
- J1 pad 19: /[1] HAT Interface/GPIO10/SPI0.MOSI -> /GPIO10/SPI0.MOSI
- J1 pad 21: /[1] HAT Interface/GPIO9/SPI0.MISO -> /GPIO9/SPI0.MISO
- J1 pad 23: /[1] HAT Interface/GPIO11/SPI0.SCLK -> /GPIO11/SPI0.SCLK
- J1 pad 26: /[1] HAT Interface/GPIO7/SPI0.CE1 -> /GPIO7/SPI0.CE1
- J1 pad 27: /[1] HAT Interface/ID_SDA -> /ID_SDA
- J1 pad 28: /[1] HAT Interface/ID_SCL -> /ID_SCL
- J1 pad 29: /[1] HAT Interface/GPIO5 -> /GPIO5
- J1 pad 3: /[1] HAT Interface/GPIO2/SDA1 -> /GPIO2/SDA1
- J1 pad 31: /[1] HAT Interface/GPIO6 -> /GPIO6
- J1 pad 32: /[1] HAT Interface/GPIO12/PWM0 -> /GPIO12/PWM0
- J1 pad 33: /[1] HAT Interface/GPIO13/PWM1 -> /GPIO13/PWM1
- J1 pad 35: /[1] HAT Interface/GPIO19/PCM.FS -> /GPIO19/PCM.FS
- J1 pad 5: /[1] HAT Interface/GPIO3/SCL1 -> /GPIO3/SCL1
Routing:
- net /[1] HAT Interface/GPIO19/PCM.FS: track 71.3 -> 0.00 mm, vias 3 -> 0
- net /[1] HAT Interface/GPIO6: track 70.9 -> 0.00 mm, vias 1 -> 0
- net /[1] HAT Interface/GPIO5: track 67.8 -> 0.00 mm, vias 3 -> 0
- net /[1] HAT Interface/GPIO27: track 63.7 -> 0.00 mm, vias 2 -> 0
- net /[1] HAT Interface/GPIO3/SCL1: track 59.6 -> 0.00 mm
- net /[1] HAT Interface/GPIO2/SDA1: track 59.3 -> 0.00 mm
- net /[1] HAT Interface/GPIO17: track 53.5 -> 0.00 mm, vias 4 -> 0
- net /[1] HAT Interface/GPIO7/SPI0.CE1: track 44.6 -> 0.00 mm
- net /[1] HAT Interface/GPIO12/PWM0: track 44.6 -> 0.00 mm
- net /[4] Motors/[4b] Servo Motor Driver/PWM A0: track 43.4 -> 0.00 mm
- net /[4] Motors/[4b] Servo Motor Driver/PWM A1: track 40.2 -> 0.00 mm
- net /[1] HAT Interface/GPIO11/SPI0.SCLK: track 37.9 -> 0.00 mm
- net /[1] HAT Interface/GPIO9/SPI0.MISO: track 37.5 -> 0.00 mm
- net /[4] Motors/[4b] Servo Motor Driver/PWM A2: track 36.7 -> 0.00 mm
- net /[4] Motors/[4b] Servo Motor Driver/PWM A5: track 36.3 -> 0.00 mm, vias 4 -> 0
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Other:
- outline, holes or cut-outs redrawn
- board text added: "CAMERA (OPTIONAL)"
- board text removed: "CPU Fan"
- board text removed: "DC Motors"
- board text removed: "Left"
- board text removed: "LiDAR Scanner"
- board text removed: "PWM Config"
- board text removed: "Right"
- board text removed: "Write Lock"

Commit message: feat: basic PCB design??? i guess?
Parts:
- added C1: 100n, Capacitor_SMD:C_0805_2012Metric, F.Cu at (108.5, 94.6)
- added D1: D, Diode_SMD:D_SOD-323F, F.Cu at (67.5, 44.0)
- added H1: MountingHole, MountingHole:MountingHole_2.2mm_M2, F.Cu at (54.6, 51.1)
- added H2: MountingHole, MountingHole:MountingHole_2.2mm_M2, F.Cu at (54.6, 57.1)
- added H3: MountingHole, MountingHole:MountingHole_2.2mm_M2, F.Cu at (54.6, 63.0)
- added H4: MountingHole, MountingHole:MountingHole_2.2mm_M2, F.Cu at (54.6, 69.0)
- added J10: Conn_01x04, Connector_PinHeader_2.54mm:PinHeader_1x04_P2.54mm_Vertical, F.Cu at (103.5, 56.5)
- added J16: Conn_02x03_Counter_Clockwise, Connector_PinHeader_2.54mm:PinHeader_2x03_P2.54mm_Vertical, F.Cu at (124.2, 92.0)
- added J2: Conn_01x02, Connector_PinSocket_2.54mm:PinSocket_1x02_P2.54mm_Vertical, F.Cu at (62.5, 44.5)
- added J3: Conn_01x02, Connector_PinSocket_2.54mm:PinSocket_1x02_P2.54mm_Vertical, F.Cu at (162.2, 78.5)
- added J4: Conn_01x02, Connector_PinSocket_2.54mm:PinSocket_1x02_P2.54mm_Vertical, F.Cu at (162.3, 69.8)
- added J5: Conn_01x02, Connector_PinSocket_2.54mm:PinSocket_1x02_P2.54mm_Vertical, F.Cu at (162.2, 91.0)
- added J6: Conn_01x02, Connector_PinSocket_2.54mm:PinSocket_1x02_P2.54mm_Vertical, F.Cu at (162.3, 82.5)
- added J7: Conn_01x04, Connector_PinHeader_2.54mm:PinHeader_1x04_P2.54mm_Vertical, F.Cu at (102.5, 66.9)
- added J8: Conn_01x02, Connector_PinSocket_2.54mm:PinSocket_1x02_P2.54mm_Vertical, F.Cu at (102.8, 80.2)
- added J9: Conn_01x04, Connector_PinHeader_2.54mm:PinHeader_1x04_P2.54mm_Vertical, F.Cu at (103.5, 53.1)
- added JP1: ID_WP, Jumper:SolderJumper-2_P1.3mm_Open_RoundedPad1.0x1.5mm, F.Cu at (119.5, 96.8)
- added Q1: SS8050, Package_TO_SOT_SMD:SOT-23, F.Cu at (70.5, 47.6)
- added R1: 3.9k, Resistor_SMD:R_1206_3216Metric, F.Cu at (110.0, 90.7)
- added R10: R, Resistor_SMD:R_0805_2012Metric, F.Cu at (66.5, 49.5)
- added R2: 3.9k, Resistor_SMD:R_1206_3216Metric, F.Cu at (116.5, 90.7)
- added U1: CAT24C256, Package_SO:SOIC-8_3.9x4.9mm_P1.27mm, F.Cu at (113.5, 95.7)
- added U2: ICM-20948, Sensor_Motion:InvenSense_QFN-24_3x3mm_P0.4mm, F.Cu at (68.9, 68.2)
- added U3: TXS0104EPW, Package_SO:TSSOP-14_4.4x5mm_P0.65mm, F.Cu at (61.9, 63.7)
- added U5: TB6612FNG, Package_SO:SSOP-24_5.3x8.2mm_P0.65mm, F.Cu at (152.1, 84.5)
- added U6: TB6612FNG, Package_SO:SSOP-24_5.3x8.2mm_P0.65mm, F.Cu at (152.2, 93.7)
- added U7: MAX98357A, Package_DFN_QFN:TQFN-16-1EP_3x3mm_P0.5mm_EP1.23x1.23mm, F.Cu at (109.8, 81.5)
Connections:
- net /GPIO14/TXD0 renamed /[1] HAT Interface/GPIO14/TXD0
- net /GPIO18/PCM.CLK renamed /[1] HAT Interface/GPIO18/PCM.CLK
- net /GPIO19/PCM.FS renamed /[1] HAT Interface/GPIO19/PCM.FS
- net /GPIO20/PCM.DIN renamed /[1] HAT Interface/GPIO20/PCM.DIN
- net /GPIO21/PCM.DOUT renamed /[1] HAT Interface/GPIO21/PCM.DOUT
- net /GPIO23 renamed /[1] HAT Interface/GPIO23
- net /GPIO24 renamed /[1] HAT Interface/GPIO24
- net /GPIO25 renamed /[1] HAT Interface/GPIO25
- net /GPIO4/GPCLK0 renamed /[1] HAT Interface/GPIO4/GPCLK0
- net /GPIO7/SPI0.CE1 renamed /[1] HAT Interface/GPIO7/SPI0.CE1
- net /GPIO8/SPI0.CE0 renamed /[1] HAT Interface/GPIO8/SPI0.CE0
- J1 pad 10: /GPIO15/RXD0 -> /[1] HAT Interface/GPIO15/RXD0
- J1 pad 11: /GPIO17 -> /[1] HAT Interface/GPIO17
- J1 pad 13: /GPIO27 -> /[1] HAT Interface/GPIO27
- J1 pad 15: /GPIO22 -> /[1] HAT Interface/GPIO22
- J1 pad 19: /GPIO10/SPI0.MOSI -> /[1] HAT Interface/GPIO10/SPI0.MOSI
- J1 pad 21: /GPIO9/SPI0.MISO -> /[1] HAT Interface/GPIO9/SPI0.MISO
- J1 pad 23: /GPIO11/SPI0.SCLK -> /[1] HAT Interface/GPIO11/SPI0.SCLK
- J1 pad 27: /ID_SDA -> /[1] HAT Interface/ID_SDA
- J1 pad 28: /ID_SCL -> /[1] HAT Interface/ID_SCL
- J1 pad 29: /GPIO5 -> /[1] HAT Interface/GPIO5
- J1 pad 3: /GPIO2/SDA1 -> /[1] HAT Interface/GPIO2/SDA1
- J1 pad 31: /GPIO6 -> /[1] HAT Interface/GPIO6
- J1 pad 32: /GPIO12/PWM0 -> /[1] HAT Interface/GPIO12/PWM0
- J1 pad 33: /GPIO13/PWM1 -> /[1] HAT Interface/GPIO13/PWM1
- J1 pad 36: /GPIO16 -> /[1] HAT Interface/GPIO16
- J1 pad 37: /GPIO26 -> /[1] HAT Interface/GPIO26
- J1 pad 5: /GPIO3/SCL1 -> /[1] HAT Interface/GPIO3/SCL1
Routing:
- net /[4] Motors/[4a] Main Motor Driver/MOTOR 2A: track 0.00 -> 15.9 mm
- net /[4] Motors/[4a] Main Motor Driver/MOTOR 2B: track 0.00 -> 15.6 mm
- net /[4] Motors/[4a] Main Motor Driver/MOTOR 1B: track 0.00 -> 14.1 mm
- net /[4] Motors/[4a] Main Motor Driver/MOTOR 1A: track 0.00 -> 13.0 mm
- net /[4] Motors/[4a] Main Motor Driver/MOTOR 4A: track 0.00 -> 12.2 mm
- net /[4] Motors/[4a] Main Motor Driver/MOTOR 4B: track 0.00 -> 12.1 mm
- net /[4] Motors/[4a] Main Motor Driver/MOTOR 3A: track 0.00 -> 11.5 mm
- net /[4] Motors/[4a] Main Motor Driver/MOTOR 3B: track 0.00 -> 9.90 mm
- net /[1] HAT Interface/ID_SDA: track 0.00 -> 9.35 mm
- net /[1] HAT Interface/ID_SCL: track 0.00 -> 7.09 mm
- net Net-(JP1-A): track 0.00 -> 4.54 mm
- net GND: track 0.00 -> 4.29 mm, vias 0 -> 1
- net /[1] HAT Interface/GPIO13/PWM1: track 0.00 -> 0.87 mm
- added copper zone on F.Cu, net +3V3
- added copper zone on B.Cu, net GND
- added copper zone on In1.Cu, net GND
Other:
- outline, holes or cut-outs redrawn
- copper layers 2 -> 4
- board text added: "DC Motors"
- board text added: "Distance Sensors"
- board text added: "LiDAR"
- board text added: "MIC IN"
- board text removed: "CAMERA (OPTIONAL)"
- board text removed: "DISPLAY (OPTIONAL)"
- board text removed: "Extend PCB edge 0.5mm if using SMT header"

Commit message: feat: semi-finalized PCB design
Parts:
- H1, H2, H3, H4: footprint MountingHole:MountingHole_2.2mm_M2 -> MountingHole:MountingHole_3.2mm_M3
- J3, J4, J5, J6, J8: footprint Connector_PinSocket_2.54mm:PinSocket_1x02_P2.54mm_Vertical -> Connector_PinHeader_2.54mm:PinHeader_1x02_P2.54mm_Vertical
- moved H3 87.5 mm to (140.5, 79.5)
- moved H1 86.0 mm to (140.5, 54.7)
- moved H4 61.4 mm to (115.1, 79.5)
- moved H2 60.7 mm to (115.2, 54.7)
- moved JP1 60.6 mm to (161.3, 53.0), turned to 180 degrees
- moved J5 59.4 mm to (103.5, 82.2), turned to 0 degrees
- moved J6 59.4 mm to (103.5, 91.0), turned to 180 degrees
- moved U1 59.3 mm to (160.1, 59.0), turned to 90 degrees
- moved C1 59.1 mm to (159.0, 64.0), turned to 0 degrees
- moved R1 53.2 mm to (155.1, 62.5), turned to 90 degrees
- moved R2 51.9 mm to (155.1, 56.0), turned to -90 degrees
- moved U6 39.4 mm to (113.0, 89.8), turned to 0 degrees
- moved J7 35.1 mm to (119.2, 97.8), turned to 90 degrees
- moved J8 34.6 mm to (132.8, 97.5), turned to 90 degrees
- moved U7 25.8 mm to (134.0, 90.5), turned to -45 degrees
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Connections:
- net /[4] Motors/[4a] Main Motor Driver/MOTOR 1A renamed Net-(J3-Pin_1)
- net /[4] Motors/[4a] Main Motor Driver/MOTOR 1B renamed Net-(J3-Pin_2)
- net /[4] Motors/[4a] Main Motor Driver/MOTOR 2A renamed Net-(J4-Pin_1)
- net /[4] Motors/[4a] Main Motor Driver/MOTOR 2B renamed Net-(J4-Pin_2)
- net /[4] Motors/[4a] Main Motor Driver/MOTOR 3A renamed Net-(J5-Pin_1)
- net /[4] Motors/[4a] Main Motor Driver/MOTOR 3B renamed Net-(J5-Pin_2)
- net /[4] Motors/[4a] Main Motor Driver/MOTOR 4A renamed Net-(J6-Pin_1)
- net /[4] Motors/[4a] Main Motor Driver/MOTOR 4B renamed Net-(J6-Pin_2)
- J16 pad 2: /[3] Fan & Sensor Systems/AUDIO CLK -> /[1] HAT Interface/GPIO18/PCM.CLK
- J16 pad 3: /[3] Fan & Sensor Systems/AUDIO FRAME -> /[1] HAT Interface/GPIO19/PCM.FS
- J16 pad 4: /[3] Fan & Sensor Systems/AUDIO IN -> /[1] HAT Interface/GPIO20/PCM.DIN
- U7 pad 1: /[3] Fan & Sensor Systems/AUDIO OUT -> /[1] HAT Interface/GPIO21/PCM.DOUT
- U7 pad 14: /[3] Fan & Sensor Systems/AUDIO FRAME -> /[1] HAT Interface/GPIO19/PCM.FS
- U7 pad 16: /[3] Fan & Sensor Systems/AUDIO CLK -> /[1] HAT Interface/GPIO18/PCM.CLK
Routing:
- net Net-(J4-Pin_1): track 15.9 -> 0.00 mm
- net Net-(J4-Pin_2): track 15.6 -> 0.00 mm
- net Net-(J3-Pin_2): track 14.1 -> 0.00 mm
- net /[1] HAT Interface/GPIO19/PCM.FS: track 0.00 -> 13.6 mm
- net Net-(J3-Pin_1): track 13.0 -> 0.00 mm
- net Net-(J6-Pin_1): track 12.2 -> 0.00 mm
- net Net-(J6-Pin_2): track 12.1 -> 0.00 mm
- net Net-(J5-Pin_1): track 11.5 -> 0.00 mm
- net /[1] HAT Interface/GPIO18/PCM.CLK: track 0.00 -> 10.4 mm
- net Net-(J5-Pin_2): track 9.90 -> 0.00 mm
- net /[3] Fan & Sensor Systems/OUT+: track 0.00 -> 6.18 mm
- net /[3] Fan & Sensor Systems/OUT-: track 0.00 -> 6.01 mm
- net /[1] HAT Interface/GPIO13/PWM1: track 0.87 -> 0.00 mm
Other:
- outline, holes or cut-outs redrawn
- board text added: "A. Left"
- board text added: "A. Right"
- board text added: "Aft DC Motors"
- board text added: "As he fell into the Icarian Sea, Icarus laughed in joy. Should he have heeded his father Daedalus' warnings, he would have lived in regret of what could have been"
- board text added: "Audio In"
- board text added: "Audio Out"
- board text added: "CPU Fan"
- board text added: "F. Left"
- board text added: "F. Right"
- board text added: "Fore DC Motors"
- board text added: "To take what is impossible, and to breathe life onto it regardless"
- board text removed: "DC Motors"
- board text removed: "MIC IN"

Commit message: feat: nets and stuff?? I guess?
I don't really remember what this commit changes
Parts:
- removed H1, H2, H3, H4: MountingHole, MountingHole:MountingHole_3.2mm_M3
- added J17: Conn_02x03_Counter_Clockwise, Connector_PinHeader_2.54mm:PinHeader_2x03_P2.54mm_Vertical, F.Cu at (148.9, 97.5)
- moved J2 86.1 mm to (147.5, 58.0), turned to 180 degrees
- moved R10 77.1 mm to (143.5, 53.0), turned to 0 degrees
- moved D1 76.4 mm to (142.5, 58.5), turned to 180 degrees
- moved Q1 69.5 mm to (139.6, 54.9), turned to -90 degrees
- moved U3 68.9 mm to (130.9, 64.7), turned to 180 degrees
- moved J3 59.9 mm to (103.0, 82.2), turned to 0 degrees
- moved J6 59.9 mm to (162.5, 80.7), turned to 0 degrees
- moved J4 59.6 mm to (103.0, 88.5)
- moved J5 59.2 mm to (162.5, 87.3)
- moved U2 53.5 mm to (123.2, 65.1), turned to -135 degrees
- moved U5 41.5 mm to (112.5, 87.5), turned to 0 degrees
- moved U6 40.9 mm to (153.0, 81.5), turned to 180 degrees
Connections:
- net Net-(J3-Pin_1) renamed /[4] Motors/MOTOR A1
- net Net-(J3-Pin_2) renamed /[4] Motors/MOTOR A2
- net Net-(J4-Pin_1) renamed /[4] Motors/MOTOR B1
- net Net-(J4-Pin_2) renamed /[4] Motors/MOTOR B2
- net Net-(J5-Pin_1) renamed /[4] Motors/MOTOR C1
- net Net-(J5-Pin_2) renamed /[4] Motors/MOTOR C2
- net Net-(J6-Pin_1) renamed /[4] Motors/MOTOR D1
- net Net-(J6-Pin_2) renamed /[4] Motors/MOTOR D2
- J16 pad 5: +5V -> +3.3V
- U7 pad 7: Net-(U7-VDD-Pad7) -> +5V
- U7 pad 8: Net-(U7-VDD-Pad7) -> +5V
Routing:
- net /[1] HAT Interface/ID_SCL: track 7.09 -> 8.88 mm
- net /[1] HAT Interface/ID_SDA: track 9.35 -> 10.8 mm
- added copper zone on In2.Cu, net GND
- removed copper zone on B.Cu, net GND
Other:
- outline, holes or cut-outs redrawn
- board text added: "LEFT"
- board text added: "RIGHT"
- board text removed: "CPU Fan"
